File: kicad-files/mana-board-kicad.kicad_pcb (KiCad board)
At the start: 2 copper layers, 200 x 125 mm, 63 parts, among them U1 Pico, U2 74AHCT1G125

Commit message: reasign capacitor numbers
Parts:
- renumbered C11 to C10, C12 to C11, C13 to C12, C14 to C13, C3 to C14, C4 to C3, C5 to C4, C6 to C5, C7 to C6, C8 to C7, C9 to C8, C10 to C9
Changed lines of the file:
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@@
     (property "ki_keywords" "capacitor cap")
     (attr smd)
-    (fp_text reference "C4" (at -0.106917 -1.883915 150) (layer "B.SilkS")
+    (fp_text reference "C3" (at -0.106917 -1.883915 150) (layer "B.SilkS")
         (effects (font (size 1 1) (thickness 0.15)) (justify mirror))
     )
@@
     (property "ki_keywords" "capacitor cap")
     (attr smd)
-    (fp_text reference "C6" (at -0.034312 -1.914382 30) (layer "B.SilkS")
+    (fp_text reference "C5" (at -0.034312 -1.914382 30) (layer "B.SilkS")
         (effects (font (size 1 1) (thickness 0.15)) (justify mirror))
     )
@@
     (property "ki_keywords" "capacitor cap")
     (attr smd)
-    (fp_text reference "C13" (at -0.01314 -2.04724 30) (layer "B.SilkS")
+    (fp_text reference "C12" (at -0.01314 -2.04724 30) (layer "B.SilkS")
         (effects (font (size 1 1) (thickness 0.15)) (justify mirror))
     )
@@
     (property "ki_keywords" "capacitor cap")
     (attr smd)
-    (fp_text reference "C14" (at 0.103001 -1.776214 30) (layer "B.SilkS")
+    (fp_text reference "C13" (at 0.103001 -1.776214 30) (layer "B.SilkS")
         (effects (font (size 1 1) (thickness 0.15)) (justify mirror))
     )
@@
     (property "ki_keywords" "capacitor cap")
     (attr smd)
-    (fp_text reference "C10" (at -0.069566 -1.853321 30) (layer "B.SilkS")
+    (fp_text reference "C9" (at -0.069566 -1.853321 30) (layer "B.SilkS")
         (effects (font (size 1 1) (thickness 0.15)) (justify mirror))
     )
@@
     (property "ki_keywords" "capacitor cap")
     (attr smd)
-    (fp_text reference "C7" (at -0.034312 -1.914382 30) (layer "B.SilkS")
+    (fp_text reference "C6" (at -0.034312 -1.914382 30) (layer "B.SilkS")
         (effects (font (size 1 1) (thickness 0.15)) (justify mirror))
     )
@@
     (property "ki_keywords" "capacitor cap")
     (attr smd)
-    (fp_text reference "C11" (at 0.083003 -1.816307 30) (layer "B.SilkS")
+    (fp_text reference "C10" (at 0.083003 -1.816307 30) (layer "B.SilkS")
         (effects (font (size 1 1) (thickness 0.15)) (justify mirror))
     )
@@
     (property "ki_keywords" "capacitor cap")
     (attr smd)
-    (fp_text reference "C8" (at 0.032205 -1.92705 30) (layer "B.SilkS")
+    (fp_text reference "C7" (at 0.032205 -1.92705 30) (layer "B.SilkS")
         (effects (font (size 1 1) (thickness 0.15)) (justify mirror))
     )
@@
     (property "ki_keywords" "capacitor cap")
     (attr smd)
-    (fp_text reference "C9" (at 0.113621 -1.766796 30) (layer "B.SilkS")
+    (fp_text reference "C8" (at 0.113621 -1.766796 30) (layer "B.SilkS")
         (effects (font (size 1 1) (thickness 0.15)) (justify mirror))
     )
@@
     (property "ki_keywords" "capacitor cap")
     (attr smd)
-    (fp_text reference "C5" (at 0.045651 -1.920928 150) (layer "B.SilkS")
+    (fp_text reference "C4" (at 0.045651 -1.920928 150) (layer "B.SilkS")
         (effects (font (size 1 1) (thickness 0.15)) (justify mirror))
     )
@@
     (property "ki_keywords" "capacitor cap")
     (attr smd)
-    (fp_text reference "C3" (at -0.008975 -2.015544 150) (layer "B.SilkS")
+    (fp_text reference "C14" (at -0.008975 -2.015544 150) (layer "B.SilkS")
         (effects (font (size 1 1) (thickness 0.15)) (justify mirror))
     )
@@
     (property "ki_keywords" "capacitor cap")
     (attr smd)
-    (fp_text reference "C12" (at -0.003049 -1.865989 30) (layer "B.SilkS")
-        (effects (font (size 1 1) (thickness 0.15)) (justify mirror))
-    )
+    (fp_text reference "C11" (at -0.003049 -1.865989 30) (layer "B.SilkS")
+        (effects (font (size 1 1) (thickness 0.15)) (justify mirror))
+    )
